File: ELED-350R1/ELED-350R1/ELED-350R1.sch (KiCad schematic (older format))
At the start: 14 parts

Commit message: symbol added
added first symbol
Parts:
- removed D? (x7): LED, symbol Device:LED
- added C1, C2, C3, C4: C, symbol Device:C
- added D10, D12, D14, D2, D4, D6, D8: LED, symbol Device:LED
- added R1, R10, R11, R2, R3, R4, R5, R6, R7, R8, R9: R, symbol Device:R
- added U1, U2: STCS2A, symbol DTL_Symbols:STCS2A
- gave numbers to parts that had none: 7
Connections:
- net labels added: +24V, +5V, D2, D3, D6, D7, D8, GND
- wire segments 0 -> 95

Commit message: Added R2
Parts:
- added C1, C10, C2, C3, C4, C5, C6, C8, C9: C, Capacitors_SMD:C_0603, symbol Device:C
- added C11, C7: CP, Capacitors_Tantalum_SMD:CP_Tantalum_Case-A_EIA-3216-18_Reflow, symbol Device:CP
- added D1, D3, D4, D6: D_Zener, Diodes_SMD:D_SOD-123, symbol Device:D_Zener
- added D2: D_TVS, Diodes_SMD:D_SMC, symbol Device:D_TVS
- added D5, D7: LED, LEDs:LED_0603, symbol Device:LED
- added J1: Screw_Terminal_01x06, DTL - KICad - Footprint:SPT-SMD 6 Pos Terminal, symbol Connector:Screw_Terminal_01x06
- added J3: AVR-ISP-6, Pin_Headers:Pin_Header_Straight_2x03_Pitch2.54mm_SMD, symbol Connector:AVR-ISP-6
- added JP1, JP2, JP3, JP4: (no value), DTL - KICad - Footprint:SolderJumper-2_P1.3mm_Open_TrianglePad1.0x1.5mm, symbol Jumper:SolderJumper_2_Open
- added JP5, JP6: Jumper, Resistors_SMD:R_2512, symbol Device:Jumper
- added Q1: IPB057N06N, TO_SOT_Packages_SMD:TO-263-3_TabPin2, symbol Device:Q_NMOS_GDS
- added R1, R2, R3, R4, R5, R6, R9: R, Resistors_SMD:R_0603, symbol Device:R
- added R16, R17, R18, R19: R, Resistors_SMD:R_1210, symbol Device:R
- added SW1: SW_Push, Buttons_Switches_SMD:SW_SPST_B3S-1100, symbol Switch:SW_Push
- added TH1: Thermistor_PTC, Resistors_SMD:R_1210, symbol Device:Thermistor_PTC
- added TP1, TP2: TestPoint, SMD_Packages:1Pin, symbol Connector:TestPoint
- added U1: LM74610-Q1, DTL - KICad - Footprint:VSSOP-8, symbol DTL_Symbols:LM74610-Q1
- added U2: ATtiny1634-SU, DTL - KICad - Footprint:ATTINY1634-SUR, symbol MCU_Microchip_ATtiny:ATtiny1634-SU
- added U3: L7805CD2T-TR, TO_SOT_Packages_SMD:TO-263-3_TabPin2, symbol Regulator_Linear:uA7805
- added Y1: Resonator, DTL - KICad - Footprint:AWSCR-CV, symbol Device:Resonator
- C12: renamed from C1; footprint (none) -> Capacitors_SMD:C_0603
- C13: renamed from C2; footprint (none) -> Capacitors_SMD:C_0603
- C14: renamed from C3; footprint (none) -> Capacitors_SMD:C_0603
- C15: renamed from C4; footprint (none) -> Capacitors_SMD:C_0603
- D10: renamed from D3; footprint (none) -> DTL - KICad - Footprint:Cree XD16
- D11: renamed from D4; footprint (none) -> DTL - KICad - Footprint:Cree XD16
- D12: renamed from D5; footprint (none) -> DTL - KICad - Footprint:Cree XD16
- D13: renamed from D6; footprint (none) -> DTL - KICad - Footprint:Cree XD16
- D14: renamed from D7; footprint (none) -> DTL - KICad - Footprint:Cree XD16
- D15: renamed from D8; footprint (none) -> DTL - KICad - Footprint:Cree XD16
- D16: renamed from D9; footprint (none) -> DTL - KICad - Footprint:Cree XD16
- D17: renamed from D10; footprint (none) -> DTL - KICad - Footprint:Cree XD16
- D18: renamed from D11; footprint (none) -> DTL - KICad - Footprint:Cree XD16
- D19: renamed from D12; footprint (none) -> DTL - KICad - Footprint:Cree XD16
- D20: renamed from D13; footprint (none) -> DTL - KICad - Footprint:Cree XD16
- D21: renamed from D14; footprint (none) -> DTL - KICad - Footprint:Cree XD16
- D8: renamed from D1; footprint (none) -> DTL - KICad - Footprint:Cree XD16
- D9: renamed from D2; footprint (none) -> DTL - KICad - Footprint:Cree XD16
- R10: renamed from R1; footprint (none) -> Resistors_SMD:R_0603
- R11: renamed from R2; footprint (none) -> Resistors_SMD:R_0603
- R12: renamed from R3; footprint (none) -> Resistors_SMD:R_0603
- R13: renamed from R4; footprint (none) -> Resistors_SMD:R_0603
- R14: renamed from R5; footprint (none) -> Resistors_SMD:R_0603
- R15: renamed from R6; footprint (none) -> Resistors_SMD:R_0603
- R20: renamed from R9; footprint (none) -> Resistors_SMD:R_0603
- R21: renamed from R10; footprint (none) -> Resistors_SMD:R_1210
- R22: renamed from R11; footprint (none) -> Resistors_SMD:R_1210
- R7, R8: footprint (none) -> Resistors_SMD:R_0603
- U4: renamed from U1; footprint (none) -> DTL - KICad - Footprint:PowerSO-10
- U5: renamed from U2; footprint (none) -> DTL - KICad - Footprint:PowerSO-10
Connections:
- net labels added: A0, A8, A9, D11, Vsup
- wire segments 95 -> 285
