File: ATmega2560 - CORE/ATmega2560 - CORE.sch (KiCad schematic (older format))
At the start: 19 parts

Commit message: Added air-speed control to lib
Connections:
- net labels added: DTR
- wire segments 185 -> 186
Changed lines of the file:
@@
 EESchema Schematic File Version 4
+LIBS:ATmega2560 - CORE-cache
 EELAYER 26 0
 EELAYER END
@@
 Wire Wire Line
 	11600 5650 11250 5650
+Text GLabel 3200 4200 2    50   Input ~ 0
+DTR
+Wire Wire Line
+	3200 4200 2950 4200
+Connection ~ 2950 4200
 $EndSCHEMATC
